Commit message: Updated joint types to continuous and prismatic

File: ros2_rolling/URDF/my_robot.urdf (robot description, URDF)
Before this commit: robot my_robot, 2 links, 1 joints
Links:
- added link third_link; visual box size=0.1 0.1 0.1
- link second_link: geometry visual cylinder length=0.2 radius=0.2
Joints:
- added joint second_third_joint: type prismatic, parent second_link, child third_link, origin xyz=0 0 0.2 rpy=0 0 0, axis 1 0 0, limit lower=-0.1 upper=0.1 effort=100 velocity=100
- joint base_second_joint: axis (none) -> 0 0 1; type fixed -> continuous
